File: Hardware/ORCA-BOARD.kicad_sch (KiCad schematic)
At the start: 22 parts, among them J1 USB_C_Receptacle_USB2.0_16P, SW1 RESET1, SW2 BOOT, U1 D3V3XA4B10LP, U2 ESP32-S3-WROOM-1, U3 AMS1117-3.3, U4 TCA9548APWR

Commit message: Subsheet de driver completado
Parts:
- added J3: Screw_Terminal_01x02, symbol Connector:Screw_Terminal_01x02
Connections:
- net DRV1_PMode: now reaches U2.22 (IO14)
- net DRV1_IN2: now reaches U2.8 (IO15)
- net DRV1_IN1: now reaches U2.9 (IO16)
- new net Driver/OUT1: J3.1 (Pin_1)
- new net Driver/OUT2: J3.2 (Pin_2)
Other:
- added sheet Driver (Driver.kicad_sch)
