File: Hardware/Driver.kicad_sch (KiCad schematic)
At the start: 8 parts, among them U5 DRV8874PWPR

Commit message: Version preeliminar blockeada Rev A PCB Control
Parts:
- R9: value 3.92k -> 2.4k
- renumbered C10_Bulk to C10_Bulk2
Connections:
- net VM renamed VMout
Other:
- note added: "Drivers-1"
- company: (none) -> L.A.A, J.F.A, F.G
- title: (none) -> ORCA BOARD
Changed lines of the file:
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@@
 	(generator_version "10.0")
 	(paper "A4")
+	(title_block
+		(title "ORCA BOARD")
+		(date "2026-08-27")
+		(rev "V.1.0.0")
+		(company "L.A.A, J.F.A, F.G")
+		(comment 1 "Felipe Gutiérrez Apráez")
+		(comment 2 "Juan Felipe Ángulo")
+		(comment 3 "Luis Ángel Aristizabal")
+	)
+	(text "Drivers-1\n"
+		(exclude_from_sim no)
+		(at 58.166 23.114 0)
+		(effects
+			(font
+				(size 12.7 12.7)
+			)
+		)
+	)
 	(junction
 		(at 101.6 87.63)
@@
 	(wire
 		(pts
+			(xy 161.29 63.5) (xy 158.75 63.5)
+		)
+		(stroke
+			(width 0)
+			(type default)
+		)
+	)
+	(wire
+		(pts
 			(xy 193.04 85.09) (xy 201.93 85.09)
 		)
@@
 	(wire
 		(pts
-			(xy 100.33 95.25) (xy 116.84 95.25)
+			(xy 113.03 95.25) (xy 116.84 95.25)
 		)
 		(stroke
@@
 	(wire
 		(pts
+			(xy 148.59 63.5) (xy 151.13 63.5)
+		)
+		(stroke
+			(width 0)
+			(type default)
+		)
+	)
+	(wire
+		(pts
 			(xy 152.4 82.55) (xy 167.64 82.55)
 		)
@@
 		)
 	)
+	(wire
+		(pts
+			(xy 161.29 62.23) (xy 161.29 63.5)
+		)
+		(stroke
+			(width 0)
+			(type default)
+		)
+	)
 	(label "CPH"
-		(at 151.13 63.5 90)
+		(at 148.59 63.5 90)
 		(effects
 			(font
@@
 	)
 	(label "CPL"
-		(at 158.75 63.5 90)
+		(at 161.29 62.23 90)
 		(effects
 			(font
@@
 			)
 		)
-		(property "Value" "VM"
+		(property "Value" "VMout"
 			(at 201.93 66.04 0)
 			(show_name no)
@@
 		(instances
 			(project "ORCA-BOARD"
+				(path "/3925f241-e926-4f70-884f-69ec72b5e7de/46317d74-6bcf-42e9-bf6a-dc4975661f21"
+					(reference "#PWR036")
+					(unit 1)
+				)
 				(path "/3925f241-e926-4f70-884f-69ec72b5e7de/6cc63822-3ea3-44ca-adf1-f22062a815da"
 					(reference "#PWR021")
@@
 		(instances
 			(project "ORCA-BOARD"
+				(path "/3925f241-e926-4f70-884f-69ec72b5e7de/46317d74-6bcf-42e9-bf6a-dc4975661f21"
+					(reference "U6")
+					(unit 1)
+				)
 				(path "/3925f241-e926-4f70-884f-69ec72b5e7de/6cc63822-3ea3-44ca-adf1-f22062a815da"
 					(reference "U5")
@@
 			)
 		)
-		(property "Value" "VM"
-			(at 170.18 68.58 0)
-			(show_name no)
-			(do_not_autoplace no)
-			(effects
-				(font
-					(size 1.27 1.27)
-				)
+		(property "Value" "VMout"
+			(at 172.72 72.3899 0)
+			(show_name no)
+			(do_not_autoplace no)
+			(effects
+				(font
+					(size 1.27 1.27)
+				)
+				(justify left)
 			)
 		)
@@
 		(instances
 			(project "ORCA-BOARD"
+				(path "/3925f241-e926-4f70-884f-69ec72b5e7de/46317d74-6bcf-42e9-bf6a-dc4975661f21"
+					(reference "#PWR034")
+					(unit 1)
+				)
 				(path "/3925f241-e926-4f70-884f-69ec72b5e7de/6cc63822-3ea3-44ca-adf1-f22062a815da"
 					(reference "#PWR020")
@@
 		(instances
 			(project "ORCA-BOARD"
+				(path "/3925f241-e926-4f70-884f-69ec72b5e7de/46317d74-6bcf-42e9-bf6a-dc4975661f21"
+					(reference "#PWR032")
+					(unit 1)
+				)
 				(path "/3925f241-e926-4f70-884f-69ec72b5e7de/6cc63822-3ea3-44ca-adf1-f22062a815da"
 					(reference "#PWR025")
@@
 		(instances
 			(project "ORCA-BOARD"
+				(path "/3925f241-e926-4f70-884f-69ec72b5e7de/46317d74-6bcf-42e9-bf6a-dc4975661f21"
+					(reference "#PWR037")
+					(unit 1)
+				)
 				(path "/3925f241-e926-4f70-884f-69ec72b5e7de/6cc63822-3ea3-44ca-adf1-f22062a815da"
 					(reference "#PWR026")
@@
 		(instances
 			(project "ORCA-BOARD"
+				(path "/3925f241-e926-4f70-884f-69ec72b5e7de/46317d74-6bcf-42e9-bf6a-dc4975661f21"
+					(reference "#PWR033")
+					(unit 1)
+				)
 				(path "/3925f241-e926-4f70-884f-69ec72b5e7de/6cc63822-3ea3-44ca-adf1-f22062a815da"
 					(reference "#PWR019")
@@
 		(instances
 			(project "ORCA-BOARD"
+				(path "/3925f241-e926-4f70-884f-69ec72b5e7de/46317d74-6bcf-42e9-bf6a-dc4975661f21"
+					(reference "R12")
+					(unit 1)
+				)
 				(path "/3925f241-e926-4f70-884f-69ec72b5e7de/6cc63822-3ea3-44ca-adf1-f22062a815da"
 					(reference "R10")
@@
 	(symbol
 		(lib_id "power:+3V3")
-		(at 100.33 95.25 0)
+		(at 113.03 95.25 90)
 		(unit 1)
 		(body_style 1)
@@
 		(in_pos_files yes)
 		(dnp no)
-		(fields_autoplaced yes)
 		(property "Reference" "#PWR023"
-			(at 100.33 99.06 0)
+			(at 116.84 95.25 0)
 			(hide yes)
 			(show_name no)
@@
 		)
 		(property "Value" "+3V3"
-			(at 100.33 90.17 0)
+			(at 113.03 97.028 90)
 			(show_name no)
 			(do_not_autoplace no)
@@
 		)
 		(property "Footprint" ""
-			(at 100.33 95.25 0)
+			(at 113.03 95.25 0)
 			(hide yes)
 			(show_name no)
@@
 		)
 		(property "Datasheet" ""
-			(at 100.33 95.25 0)
+			(at 113.03 95.25 0)
 			(hide yes)
 			(show_name no)
@@
 		)
 		(property "Description" "Power symbol creates a global label with name \"+3V3\""
-			(at 100.33 95.25 0)
+			(at 113.03 95.25 0)
 			(hide yes)
 			(show_name no)
@@
 		(instances
 			(project "ORCA-BOARD"
+				(path "/3925f241-e926-4f70-884f-69ec72b5e7de/46317d74-6bcf-42e9-bf6a-dc4975661f21"
+					(reference "#PWR029")
+					(unit 1)
+				)
 				(path "/3925f241-e926-4f70-884f-69ec72b5e7de/6cc63822-3ea3-44ca-adf1-f22062a815da"
 					(reference "#PWR023")
@@
 		(instances
 			(project "ORCA-BOARD"
+				(path "/3925f241-e926-4f70-884f-69ec72b5e7de/46317d74-6bcf-42e9-bf6a-dc4975661f21"
+					(reference "C11")
+					(unit 1)
+				)
 				(path "/3925f241-e926-4f70-884f-69ec72b5e7de/6cc63822-3ea3-44ca-adf1-f22062a815da"
 					(reference "C7")
@@
 		(instances
 			(project "ORCA-BOARD"
+				(path "/3925f241-e926-4f70-884f-69ec72b5e7de/46317d74-6bcf-42e9-bf6a-dc4975661f21"
+					(reference "C10")
+					(unit 1)
+				)
 				(path "/3925f241-e926-4f70-884f-69ec72b5e7de/6cc63822-3ea3-44ca-adf1-f22062a815da"
 					(reference "C8")
@@
 		(instances
 			(project "ORCA-BOARD"
+				(path "/3925f241-e926-4f70-884f-69ec72b5e7de/46317d74-6bcf-42e9-bf6a-dc4975661f21"
+					(reference "C12")
+					(unit 1)
+				)
 				(path "/3925f241-e926-4f70-884f-69ec72b5e7de/6cc63822-3ea3-44ca-adf1-f22062a815da"
 					(reference "C9")
@@
 		(instances
 			(project "ORCA-BOARD"
+				(path "/3925f241-e926-4f70-884f-69ec72b5e7de/46317d74-6bcf-42e9-bf6a-dc4975661f21"
+					(reference "R13")
+					(unit 1)
+				)
 				(path "/3925f241-e926-4f70-884f-69ec72b5e7de/6cc63822-3ea3-44ca-adf1-f22062a815da"
 					(reference "R11")
@@
 		(instances
 			(project "ORCA-BOARD"
+				(path "/3925f241-e926-4f70-884f-69ec72b5e7de/46317d74-6bcf-42e9-bf6a-dc4975661f21"
+					(reference "#PWR028")
+					(unit 1)
+				)
 				(path "/3925f241-e926-4f70-884f-69ec72b5e7de/6cc63822-3ea3-44ca-adf1-f22062a815da"
 					(reference "#PWR024")
@@
 		(instances
 			(project "ORCA-BOARD"
+				(path "/3925f241-e926-4f70-884f-69ec72b5e7de/46317d74-6bcf-42e9-bf6a-dc4975661f21"
+					(reference "#PWR035")
+					(unit 1)
+				)
 				(path "/3925f241-e926-4f70-884f-69ec72b5e7de/6cc63822-3ea3-44ca-adf1-f22062a815da"
 					(reference "#PWR022")
@@
 		(instances
 			(project "ORCA-BOARD"
+				(path "/3925f241-e926-4f70-884f-69ec72b5e7de/46317d74-6bcf-42e9-bf6a-dc4975661f21"
+					(reference "#PWR031")
+					(unit 1)
+				)
 				(path "/3925f241-e926-4f70-884f-69ec72b5e7de/6cc63822-3ea3-44ca-adf1-f22062a815da"
 					(reference "#PWR018")
@@
 			)
 		)
-		(property "Value" "3.92k"
+		(property "Value" "2.4k"
 			(at 171.45 84.836 90)
 			(show_name no)
@@
 		(instances
 			(project "ORCA-BOARD"
+				(path "/3925f241-e926-4f70-884f-69ec72b5e7de/46317d74-6bcf-42e9-bf6a-dc4975661f21"
+					(reference "R14")
+					(unit 1)
+				)
 				(path "/3925f241-e926-4f70-884f-69ec72b5e7de/6cc63822-3ea3-44ca-adf1-f22062a815da"
 					(reference "R9")
@@
 		(instances
 			(project "ORCA-BOARD"
+				(path "/3925f241-e926-4f70-884f-69ec72b5e7de/46317d74-6bcf-42e9-bf6a-dc4975661f21"
+					(reference "#PWR030")
+					(unit 1)
+				)
 				(path "/3925f241-e926-4f70-884f-69ec72b5e7de/6cc63822-3ea3-44ca-adf1-f22062a815da"
 					(reference "#PWR027")
@@
 		(dnp no)
 		(fields_autoplaced yes)
-		(property "Reference" "C10_Bulk"
+		(property "Reference" "C10_Bulk2"
 			(at 213.36 80.0099 0)
 			(show_name no)
@@
 		(instances
 			(project "ORCA-BOARD"
+				(path "/3925f241-e926-4f70-884f-69ec72b5e7de/46317d74-6bcf-42e9-bf6a-dc4975661f21"
+					(reference "C10_Bulk1")
+					(unit 1)
+				)
 				(path "/3925f241-e926-4f70-884f-69ec72b5e7de/6cc63822-3ea3-44ca-adf1-f22062a815da"
-					(reference "C10_Bulk")
-					(unit 1)
-				)
+					(reference "C10_Bulk2")
+					(unit 1)
+				)
